File: display.kicad_sch (KiCad schematic)
At the start: 72 parts

Commit message: Rename files and change title block
Other:
- company: Antmicro Ltd -> Capable Robot Components, Inc.
- title: Jetson Nano Baseboard -> Capable Jetson Carrier
Changed lines of the file:
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@@
   (paper "A3")
   (title_block
-    (title "Jetson Nano Baseboard")
-    (date "2022-02-04")
-    (rev "1.5.1")
-    (company "Antmicro Ltd")
-    (comment 1 "www.antmicro.com")
-    (comment 2 "Antmicro Ltd")
+    (title "Capable Jetson Carrier")
+    (date "2022-04-06")
+    (rev "v1.0")
+    (company "Capable Robot Components, Inc.")
+    (comment 1 "www.capablerobot.com")
+    (comment 2 "")
   )
   (junction (at 128.905 223.52) (diameter 0) (color 0 0 0 0)

Commit message: Rebuild
Parts:
- C1, C2, C3, C4: value (none) -> C_4u7_0402; footprint (none) -> jetson-nano-baseboard-footprints:0402-cap
- C12, C26, C27, C39, C40, C42, C43, C44, C45, C5, C6, C7, C73, C74, C75, C76, C77, C78, C79, C8, C80: value (none) -> C_100n_0402; footprint (none) -> jetson-nano-baseboard-footprints:0402-cap
- D10, D11, D12: renamed from D?; value (none) -> PESD2USB5UV-TR; footprint (none) -> jetson-nano-baseboard-footprints:SOT-23s
- D2, D4: value (none) -> 1N4148WS; footprint (none) -> jetson-nano-baseboard-footprints:SOD-323
- IC11: value (none) -> SN74LV1T125DBVR; footprint (none) -> jetson-nano-baseboard-footprints:SOT-23-5
- IC18, IC2: value (none) -> ~; footprint (none) -> jetson-nano-baseboard-footprints:SON-15
- IC6: value (none) -> PCA9517ADP; footprint (none) -> jetson-nano-baseboard-footprints:MSOP-8
- J1: value (none) -> 46756-1001; footprint (none) -> jetson-nano-baseboard-footprints:HDMI_Micro-D_Molex_46765-1x01
- J2: value (none) -> 2129320-3; footprint (none) -> jetson-nano-baseboard-footprints:2129320-3
- L10, L8, L9: value (none) -> BLM18SG121TN1D; footprint (none) -> jetson-nano-baseboard-footprints:0603
- M1: value (none) -> ~; footprint (none) -> jetson-nano-baseboard-footprints:jetson-nano-connector
- R1, R10, R2, R3, R4, R7, R8, R9: value (none) -> R_5R6_0402; footprint (none) -> jetson-nano-baseboard-footprints:0402-res
- R100, R26, R30: value (none) -> R_100k_0402; footprint (none) -> jetson-nano-baseboard-footprints:0402-res
- R11, R37, R5, R6, R81, R83, R88: value (none) -> R_2k_0402; footprint (none) -> jetson-nano-baseboard-footprints:0402-res
- R12, R82, R98, R99: value (none) -> R_0R_0402; footprint (none) -> jetson-nano-baseboard-footprints:0402-res
- R31, R32: value (none) -> R_1M0_0402; footprint (none) -> jetson-nano-baseboard-footprints:0402-res
- T1: value (none) -> BSS138APW; footprint (none) -> jetson-nano-baseboard-footprints:SC70-3
- TP2, TP25, TP26, TP33, TP34, TP35, TP36: value (none) -> ~; footprint (none) -> jetson-nano-baseboard-footprints:TP-R-1.5
