File: capable_jetson_carrier.kicad_sch (KiCad schematic)
At the start: 3 parts

Commit message: Rename files and change title block
Other:
- company: (none) -> Capable Robot Components, Inc.
- title: Jetson Nano Baseboard -> Capable Jetson Carrier
Changed lines of the file:
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@@
   (paper "A3")
   (title_block
-    (title "Jetson Nano Baseboard")
-    (date "2022-02-04")
-    (rev "1.5.1")
-    (comment 1 "www.antmicro.com")
-    (comment 2 "Antmicro Ltd")
+    (title "Capable Jetson Carrier")
+    (date "2022-04-06")
+    (rev "v1.0")
+    (company "Capable Robot Components, Inc.")
+    (comment 1 "www.capablerobot.com")
+    (comment 2 "")
   )
   (text "Text" (at 67.7926 1253.8202 0)

Commit message: Rebuild
Parts:
- N1: value (none) -> antmicro_logo; footprint (none) -> jetson-nano-baseboard-footprints:antmicro-logo_scaled_15mm
- N2: value (none) -> oshw_logo; footprint (none) -> jetson-nano-baseboard-footprints:oshw-logo
- N3: value (none) -> crc_logo; footprint (none) -> jetson-nano-baseboard-footprints:CRC_logo_15mm
Changed lines of the file:
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@@
     (company "Capable Robot Components, Inc.")
     (comment 1 "www.capablerobot.com")
-    (comment 2 "")
   )
   (text "Text" (at 67.7926 1253.8202 0)
@@
       (effects (font (size 1.27 1.27)) (justify left))
     )
-    (property "Value" "" (id 1) (at 388.9756 246.9642 0)
+    (property "Value" "antmicro_logo" (id 1) (at 388.9756 246.9642 0)
       (effects (font (size 1.27 1.27)) (justify left))
     )
-    (property "Footprint" "" (id 2) (at 381 240.665 0)
+    (property "Footprint" "jetson-nano-baseboard-footprints:antmicro-logo_scaled_15mm" (id 2) (at 381 240.665 0)
       (effects (font (size 1.27 1.27)) hide)
     )
@@
       (effects (font (size 1.27 1.27)) (justify left))
     )
-    (property "Value" "" (id 1) (at 389.1026 241.6302 0)
+    (property "Value" "oshw_logo" (id 1) (at 389.1026 241.6302 0)
       (effects (font (size 1.27 1.27)) (justify left))
     )
-    (property "Footprint" "" (id 2) (at 384.683 245.491 0)
+    (property "Footprint" "jetson-nano-baseboard-footprints:oshw-logo" (id 2) (at 384.683 245.491 0)
       (effects (font (size 1.27 1.27)) hide)
     )
@@
       (effects (font (size 1.27 1.27)) (justify left))
     )
-    (property "Value" "" (id 1) (at 389.1026 235.9152 0)
+    (property "Value" "crc_logo" (id 1) (at 389.1026 235.9152 0)
       (effects (font (size 1.27 1.27)) (justify left))
     )
-    (property "Footprint" "" (id 2) (at 384.683 239.776 0)
+    (property "Footprint" "jetson-nano-baseboard-footprints:CRC_logo_15mm" (id 2) (at 384.683 239.776 0)
       (effects (font (size 1.27 1.27)) hide)
     )
@@
       (reference "#GND_0118") (unit 1) (value "GND") (footprint "")
     )
-    (path "/00000000-0000-0000-0000-000060b0f7be/00000000-0000-0000-0000-000060d686f7"
-      (reference "#GND_0119") (unit 1) (value "GND") (footprint "")
-    )
     (path "/00000000-0000-0000-0000-00006096d016/00000000-0000-0000-0000-00005e7104e1"
       (reference "#GND_0120") (unit 1) (value "GND") (footprint "")
@@
       (reference "R131") (unit 1) (value "R_10k_0402") (footprint "jetson-nano-baseboard-footprints:0402-res")
     )
-    (path "/00000000-0000-0000-0000-000060b0f7be/00000000-0000-0000-0000-000062df2d52"
-      (reference "R132") (unit 1) (value "R_0R_0402") (footprint "jetson-nano-baseboard-footprints:0402-res")
-    )
     (path "/00000000-0000-0000-0000-0000610accab/00000000-0000-0000-0000-00005e710410"
       (reference "REC1") (unit 1) (value "~") (footprint "jetson-nano-baseboard-footprints:TL3340AF160QG")
@@
       (reference "TP29") (unit 1) (value "~") (footprint "jetson-nano-baseboard-footprints:TP-R-1.5")
     )
-    (path "/00000000-0000-0000-0000-000060b0f7be/00000000-0000-0000-0000-00005f7a644a"
-      (reference "TP30") (unit 1) (value "TC2030") (footprint "jetson-nano-baseboard-footprints:TC2030")
-    )
     (path "/00000000-0000-0000-0000-0000610accab/00000000-0000-0000-0000-00005e7103ea"

Commit message: Remove displays
Other:
- removed sheet Display

Commit message: Update symbol library to v6
Parts:
- N1: footprint jetson-nano-baseboard-footprints:antmicro-logo_scaled_15mm -> jetson-nano-baseboard-footprints:antmicro-logo
Changed lines of the file:
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@@
       (effects (font (size 1.27 1.27)) (justify left))
     )
-    (property "Footprint" "jetson-nano-baseboard-footprints:antmicro-logo_scaled_15mm" (id 2) (at 381 240.665 0)
+    (property "Footprint" "jetson-nano-baseboard-footprints:antmicro-logo" (id 2) (at 381 240.665 0)
       (effects (font (size 1.27 1.27)) hide)
     )
@@
     )
     (path "/00000000-0000-0000-0000-000060d9f63d/00000000-0000-0000-0000-0000605d7511"
-      (reference "J6") (unit 1) (value "WE_68715014522") (footprint "jetson-nano-baseboard-footprints:WE_68715014522_ONE-SIDE")
+      (reference "J6") (unit 1) (value "WE_68715014522") (footprint "jetson-nano-baseboard-footprints:WE_68715014522")
     )
     (path "/00000000-0000-0000-0000-000060d9f63d/00000000-0000-0000-0000-0000605e5dc9"
@@
     )
     (path "/00000000-0000-0000-0000-000060bdca6d"
-      (reference "N1") (unit 1) (value "antmicro_logo") (footprint "jetson-nano-baseboard-footprints:antmicro-logo_scaled_15mm")
+      (reference "N1") (unit 1) (value "antmicro_logo") (footprint "jetson-nano-baseboard-footprints:antmicro-logo")
     )
     (path "/00000000-0000-0000-0000-000060bdce33"
@@
     )
     (path "/00000000-0000-0000-0000-000060d9f63d/93adc4d8-b8ca-4365-8648-37e0ecffa5a9"
-      (reference "R12") (unit 1) (value "R_0R_0603") (footprint "jetson-nano-baseboard-footprints:0603-res")
+      (reference "R12") (unit 1) (value "R_0R_0603") (footprint "jetson-nano-baseboard-footprints:0402-res")
     )
     (path "/00000000-0000-0000-0000-000060d9f63d/a7259f25-67a2-44e4-9c1d-e531ba0e33bc"
-      (reference "R13") (unit 1) (value "R_0R_0603") (footprint "jetson-nano-baseboard-footprints:0603-res")
+      (reference "R13") (unit 1) (value "R_0R_0603") (footprint "jetson-nano-baseboard-footprints:0402-res")
     )
     (path "/00000000-0000-0000-0000-0000610accab/00000000-0000-0000-0000-000062cd1118"
@@
     )
     (path "/00000000-0000-0000-0000-0000608e1758/00000000-0000-0000-0000-00005e710438"
-      (reference "SP7") (unit 1) (value "9774040151") (footprint "jetson-nano-baseboard-footprints:9774060151")
+      (reference "SP7") (unit 1) (value "9774040151") (footprint "jetson-nano-baseboard-footprints:M2.5-4mm")
     )
     (path "/00000000-0000-0000-0000-0000610accab/00000000-0000-0000-0000-00006073683d"
