File: spi-devices.kicad_sch (KiCad schematic)
At the start: 3 parts, among them U5 IIM-42652

Commit message: Change FPGA to ICE40UP5K
Parts:
- added C89: C_1u_0603, Capacitor_SMD:C_0603_1608Metric, symbol jetson-nano-baseboard:C_100n_0402
- added R104: R_1k_0402, Resistor_SMD:R_0402_1005Metric, symbol jetson-nano-baseboard:R_10k_0402
Connections:
- net GND: now also C89.1
- net 3V3_SYS renamed 1V8_SYS
- net 1V8_SYS: now also C89.2
- net IMU-INT1: no longer names the net of U5.4 (INT1/INT)
- net IMU-INT1: now also R104.1
- new net GPIO00: R104.2
Changed lines of the file:
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@@
 (kicad_sch (version 20211123) (generator eeschema)
   (paper "A4")
-  (junction (at 87.122 29.845) (diameter 0) (color 0 0 0 0)
+  (junction (at 87.122 29.8704) (diameter 0) (color 0 0 0 0)
+  )
+  (junction (at 97.9424 29.8704) (diameter 0) (color 0 0 0 0)
   )
   (junction (at 80.772 33.02) (diameter 0) (color 0 0 0 0)
+  )
+  (junction (at 97.9424 40.64) (diameter 0) (color 0 0 0 0)
+  )
+  (junction (at 108.204 29.8704) (diameter 0) (color 0 0 0 0)
   )
   (junction (at 87.122 40.64) (diameter 0) (color 0 0 0 0)
   )
   (no_connect (at 75.692 43.18))
-  (wire (pts (xy 97.917 29.845) (xy 97.917 31.75))
+  (wire (pts (xy 97.9424 29.8704) (xy 97.9424 31.75))
     (stroke (width 0) (type default) (color 0 0 0 0))
   )
@@
     (stroke (width 0) (type default) (color 0 0 0 0))
   )
-  (wire (pts (xy 97.917 40.64) (xy 87.122 40.64))
+  (wire (pts (xy 97.9424 40.64) (xy 87.122 40.64))
     (stroke (width 0) (type default) (color 0 0 0 0))
   )
-  (wire (pts (xy 97.917 39.37) (xy 97.917 40.64))
+  (wire (pts (xy 97.9424 39.37) (xy 97.9424 40.64))
+    (stroke (width 0) (type default) (color 0 0 0 0))
+  )
+  (wire (pts (xy 97.9424 29.8704) (xy 108.204 29.8704))
     (stroke (width 0) (type default) (color 0 0 0 0))
   )
@@
     (stroke (width 0) (type default) (color 0 0 0 0))
   )
-  (wire (pts (xy 87.122 29.845) (xy 87.122 31.75))
+  (wire (pts (xy 87.122 29.8704) (xy 87.122 31.75))
     (stroke (width 0) (type default) (color 0 0 0 0))
   )
@@
     (stroke (width 0) (type default) (color 0 0 0 0))
   )
+  (wire (pts (xy 108.204 40.64) (xy 97.9424 40.64))
+    (stroke (width 0) (type default) (color 0 0 0 0))
+  )
+  (wire (pts (xy 108.204 29.8704) (xy 109.8804 29.8704))
+    (stroke (width 0) (type default) (color 0 0 0 0))
+  )
   (wire (pts (xy 45.212 38.1) (xy 52.832 38.1))
     (stroke (width 0) (type default) (color 0 0 0 0))
   )
-  (wire (pts (xy 87.122 27.94) (xy 87.122 29.845))
+  (wire (pts (xy 87.122 29.8704) (xy 97.9424 29.8704))
     (stroke (width 0) (type default) (color 0 0 0 0))
   )
-  (wire (pts (xy 87.122 29.845) (xy 97.917 29.845))
+  (wire (pts (xy 108.204 39.37) (xy 108.204 40.64))
     (stroke (width 0) (type default) (color 0 0 0 0))
   )
@@
     (stroke (width 0) (type default) (color 0 0 0 0))
   )
-  (wire (pts (xy 80.772 33.02) (xy 80.772 29.845))
+  (wire (pts (xy 80.772 33.02) (xy 80.772 29.8704))
     (stroke (width 0) (type default) (color 0 0 0 0))
   )
@@
     (stroke (width 0) (type default) (color 0 0 0 0))
   )
-  (wire (pts (xy 80.772 29.845) (xy 87.122 29.845))
+  (wire (pts (xy 80.772 29.8704) (xy 87.122 29.8704))
+    (stroke (width 0) (type default) (color 0 0 0 0))
+  )
+  (wire (pts (xy 108.204 29.8704) (xy 108.204 31.75))
     (stroke (width 0) (type default) (color 0 0 0 0))
   )
@@
     (stroke (width 0) (type default) (color 0 0 0 0))
   )
+  (wire (pts (xy 31.3944 45.72) (xy 38.1 45.72))
+    (stroke (width 0) (type default) (color 0 0 0 0))
+  )
   (wire (pts (xy 45.72 48.26) (xy 52.832 48.26))
     (stroke (width 0) (type default) (color 0 0 0 0))
   )
-  (global_label "SPI1-CIPO" (shape input) (at 45.212 33.02 180) (fields_autoplaced)
+  (global_label "SPI1-CIPO" (shape output) (at 45.212 33.02 180) (fields_autoplaced)
     (effects (font (size 1.27 1.27)) (justify right))
     (property "Intersheet References" "${INTERSHEET_REFS}" (id 0) (at 32.5464 32.9406 0)
@@
     )
   )
-  (global_label "IMU-INT1" (shape bidirectional) (at 45.72 45.72 180) (fields_autoplaced)
-    (effects (font (size 1.27 1.27)) (justify right))
-    (property "Intersheet References" "${INTERSHEET_REFS}" (id 0) (at 34.3244 45.7994 0)
-      (effects (font (size 1.27 1.27)) (justify right) hide)
-    )
-  )
-  (global_label "3V3_SYS" (shape input) (at 87.122 27.94 90) (fields_autoplaced)
-    (effects (font (size 1.27 1.27)) (justify left))
-    (property "Intersheet References" "${INTERSHEET_REFS}" (id 0) (at -160.528 -101.6 0)
-      (effects (font (size 1.27 1.27)) hide)
-    )
-  )
-  (global_label "SPI1-COPI" (shape output) (at 45.212 35.56 180) (fields_autoplaced)
+  (global_label "SPI1-COPI" (shape input) (at 45.212 35.56 180) (fields_autoplaced)
     (effects (font (size 1.27 1.27)) (justify right))
     (property "Intersheet References" "${INTERSHEET_REFS}" (id 0) (at 32.5464 35.4806 0)
@@
     )
   )
+  (global_label "1V8_SYS" (shape input) (at 109.8804 29.8704 0) (fields_autoplaced)
+    (effects (font (size 1.27 1.27)) (justify left))
+    (property "Intersheet References" "${INTERSHEET_REFS}" (id 0) (at 120.1875 29.791 0)
+      (effects (font (size 1.27 1.27)) (justify left) hide)
+    )
+  )
   (global_label "IMU-INT2" (shape bidirectional) (at 45.72 48.26 180) (fields_autoplaced)
     (effects (font (size 1.27 1.27)) (justify right))
@@
     )
   )
-  (symbol (lib_id "jetson-nano-baseboard:C_100n_0402") (at 97.917 35.56 180) (unit 1)
+  (global_label "GPIO00" (shape bidirectional) (at 31.3944 45.72 180) (fields_autoplaced)
+    (effects (font (size 1.27 1.27)) (justify right))
+    (property "Intersheet References" "${INTERSHEET_REFS}" (id 0) (at 22.1759 45.6406 0)
+      (effects (font (size 1.27 1.27)) (justify right) hide)
+    )
+  )
+  (symbol (lib_id "jetson-nano-baseboard:R_10k_0402") (at 41.91 45.72 180) (unit 1)
     (in_bom yes) (on_board yes)
-    (property "Reference" "C15" (id 0) (at 105.537 34.29 0)
+    (property "Reference" "R104" (id 0) (at 50.5714 44.6024 0)
       (effects (font (size 1.524 1.524)) (justify left))
     )
-    (property "Value" "C_100n_0402" (id 1) (at 97.917 31.75 0)
+    (property "Value" "R_1k_0402" (id 1) (at 41.91 41.91 0)
       (effects (font (size 1.524 1.524)) hide)
     )
-    (property "Footprint" "jetson-nano-baseboard-footprints:0402-cap" (id 2) (at 92.837 40.64 0)
+    (property "Footprint" "Resistor_SMD:R_0402_1005Metric" (id 2) (at 36.83 50.8 0)
       (effects (font (size 1.524 1.524)) (justify left) hide)
     )
-    (property "Datasheet" "" (id 3) (at 97.917 35.56 0)
+    (property "Datasheet" "" (id 3) (at 41.91 45.72 0)
       (effects (font (size 1.27 1.27)) hide)
     )
-    (property "Manufacturer" "Walsin" (id 4) (at 92.837 45.72 0)
+    (property "Val" "1k" (id 6) (at 43.815 45.72 0)
+      (effects (font (size 1.27 1.27)) (justify left))
+    )
+    (pin "1")
+    (pin "2")
+  )
+  (symbol (lib_id "jetson-nano-baseboard:C_100n_0402") (at 108.204 35.56 0) (mirror x) (unit 1)
+    (in_bom yes) (on_board yes)
+    (property "Reference" "C89" (id 0) (at 112.0394 33.7566 0)
+      (effects (font (size 1.524 1.524)))
+    )
+    (property "Value" "C_1u_0603" (id 1) (at 108.204 31.75 0)
+      (effects (font (size 1.524 1.524)) hide)
+    )
+    (property "Footprint" "Capacitor_SMD:C_0603_1608Metric" (id 2) (at 113.284 40.64 0)
       (effects (font (size 1.524 1.524)) (justify left) hide)
     )
-    (property "MPN" "0402X104K6R3CT" (id 5) (at 92.837 43.18 0)
+    (property "Datasheet" "" (id 3) (at 108.204 35.56 0)
+      (effects (font (size 1.27 1.27)) hide)
+    )
+    (property "Val" "1u" (id 6) (at 111.887 36.6776 0))
+    (pin "1")
+    (pin "2")
+  )
+  (symbol (lib_id "jetson-nano-baseboard:C_100n_0402") (at 97.9424 35.56 180) (unit 1)
+    (in_bom yes) (on_board yes)
+    (property "Reference" "C15" (id 0) (at 105.5624 34.29 0)
+      (effects (font (size 1.524 1.524)) (justify left))
+    )
+    (property "Value" "C_100n_0402" (id 1) (at 97.9424 31.75 0)
+      (effects (font (size 1.524 1.524)) hide)
+    )
+    (property "Footprint" "jetson-nano-baseboard-footprints:0402-cap" (id 2) (at 92.8624 40.64 0)
       (effects (font (size 1.524 1.524)) (justify left) hide)
     )
-    (property "Val" "100n" (id 6) (at 106.172 36.195 0)
+    (property "Datasheet" "" (id 3) (at 97.9424 35.56 0)
+      (effects (font (size 1.27 1.27)) hide)
+    )
+    (property "Manufacturer" "Walsin" (id 4) (at 92.8624 45.72 0)
+      (effects (font (size 1.524 1.524)) (justify left) hide)
+    )
+    (property "MPN" "0402X104K6R3CT" (id 5) (at 92.8624 43.18 0)
+      (effects (font (size 1.524 1.524)) (justify left) hide)
+    )
+    (property "Val" "100n" (id 6) (at 106.1974 36.195 0)
       (effects (font (size 1.27 1.27)) (justify left))
     )
